Commit message: Implemented Package Structure Standarization, 3D Mapping and Navigation via RTABMap(Rviz & Rtabmap_viz)

File: src/navrover_description/urdf/kinect_sensor.xacro (robot description, xacro)
@@ -48,5 +48,5 @@
      <origin xyz="0 0 0" rpy="0 0 ${PI/2}"/>
       <geometry>
-       <mesh filename="package://navrover_simulation/meshes/sensors/kinect.dae"/>
+       <mesh filename="package://navrover_description/meshes/sensors/kinect.dae"/>
       </geometry>
     </visual>

File: src/navrover_description/urdf/rover.xacro (robot description, xacro)
@@ -1,6 +1,6 @@
 <?xml version="1.0"?>
 <robot xmlns:xacro="http://www.ros.org/wiki/xacro" name="rover">
-  <xacro:include filename="$(find navrover_simulation)/urdf/rover.gazebo" />
-  <xacro:include filename="$(find navrover_simulation)/urdf/kinect_sensor.xacro" />
+  <xacro:include filename="$(find navrover_description)/urdf/rover.gazebo" />
+  <xacro:include filename="$(find navrover_description)/urdf/kinect_sensor.xacro" />
   <xacro:property name="PI" value="3.1415926535897931"/>
   <xacro:macro name="default_inertial" params="mass">
