Commit message: Update rover model colors in Gazebo simulation

File: navrover_description/urdf/navrover.xacro (robot description, xacro)
@@ -4,4 +4,6 @@
 <xacro:include filename="$(find navrover_description)/urdf/navrover.trans" />
 <xacro:include filename="$(find navrover_description)/urdf/navrover.gazebo" />
+<!--New base_footprint link -->
+<!-- <link name="base_footprint"/> -->
 <link name="base_link">
   <inertial>
@@ -244,9 +246,16 @@
   </collision>
 </link>
+<!-- <joint name="base_footprint_joint" type="fixed">
+  <origin xyz="0 0 0" rpy="0 0 0"/>
+  <parent link="base_footprint"/>
+  <child link="base_link"/>
+</joint> -->
 <joint name="right_front_wheel_joint" type="continuous">
   <origin xyz="0.003502 -0.008922 -0.079551" rpy="0 0 0"/>
   <parent link="right_front_motor_1"/>
   <child link="right_front_wheel_1"/>
-  <axis xyz="-0.0 1.0 0.0"/>
+  <axis xyz="0.0 1.0 0.0"/>
+  <limit effort="2.0" velocity="6.0"/>
+  <dynamics friction="0.3125" damping="0.1"/>
 </joint>
 <joint name="right_rear_wheel_joint" type="continuous">
@@ -254,5 +263,7 @@
   <parent link="right_rear_motor_1"/>
   <child link="right_rear_wheel_1"/>
-  <axis xyz="-0.0 1.0 0.0"/>
+  <axis xyz="0.0 1.0 0.0"/>
+  <limit effort="2.0" velocity="6.0"/>
+  <dynamics friction="0.3125" damping="0.1"/>
 </joint>
 <joint name="left_front_wheel_joint" type="continuous">
@@ -260,5 +271,7 @@
   <parent link="left_front_motor_1"/>
   <child link="left_front_wheel_1"/>
-  <axis xyz="0.0 -1.0 0.0"/>
+  <axis xyz="0.0 1.0 0.0"/>
+  <limit effort="2.0" velocity="6.0"/>
+  <dynamics friction="0.3125" damping="0.1"/>
 </joint>
 <joint name="left_front_motor_mount_joint" type="fixed">
@@ -281,5 +294,5 @@
   <parent link="base_link"/>
   <child link="right_rocker_arm_1"/>
-  <axis xyz="0.0 -1.0 -0.0"/>
+  <axis xyz="0.0 -1.0 0.0"/>
   <limit upper="0.261799" lower="-0.261799" effort="100" velocity="100"/>
 </joint>
@@ -305,5 +318,7 @@
   <parent link="left_rear_motor_1"/>
   <child link="left_rear_wheel_1"/>
-  <axis xyz="0.0 -1.0 0.0"/>
+  <axis xyz="0.0 1.0 0.0"/>
+  <limit effort="2.0" velocity="6.0"/>
+  <dynamics friction="0.3125" damping="0.1"/>
 </joint>
 </robot>

Commit message: Update rover wheel friction and collision properties in Gazebo simulation

File: navrover_description/urdf/navrover.xacro (robot description, xacro)
@@ -4,6 +4,4 @@
 <xacro:include filename="$(find navrover_description)/urdf/navrover.trans" />
 <xacro:include filename="$(find navrover_description)/urdf/navrover.gazebo" />
-<!--New base_footprint link -->
-<!-- <link name="base_footprint"/> -->
 <link name="base_link">
   <inertial>
@@ -26,64 +24,4 @@
   </collision>
 </link>
-<link name="right_front_wheel_1">
-  <inertial>
-    <origin xyz="-8.102817960486952e-07 -0.055271110065370055 4.86858583587102e-07" rpy="0 0 0"/>
-    <mass value="0.7376559494744219"/>
-    <inertia ixx="0.001132" iyy="0.001768" izz="0.001132" ixy="0.0" iyz="-0.0" ixz="-0.0"/>
-  </inertial>
-  <visual>
-    <origin xyz="-0.262818 0.165429 -0.062925" rpy="0 0 0"/>
-    <geometry>
-      <mesh filename="file://$(find navrover_description)/meshes/right_front_wheel_1.stl" scale="0.001 0.001 0.001"/>
-    </geometry>
-    <material name="silver"/>
-  </visual>
-  <collision>
-    <origin xyz="-0.262818 0.165429 -0.062925" rpy="0 0 0"/>
-    <geometry>
-      <mesh filename="file://$(find navrover_description)/meshes/right_front_wheel_1.stl" scale="0.001 0.001 0.001"/>
-    </geometry>
-  </collision>
-</link>
-<link name="right_rear_wheel_1">
-  <inertial>
-    <origin xyz="-5.274171592795085e-07 -0.0552717902856055 4.929203514525415e-07" rpy="0 0 0"/>
-    <mass value="0.737655949474422"/>
-    <inertia ixx="0.001132" iyy="0.001768" izz="0.001132" ixy="0.0" iyz="-0.0" ixz="-0.0"/>
-  </inertial>
-  <visual>
-    <origin xyz="0.245885 0.165394 -0.063543" rpy="0 0 0"/>
-    <geometry>
-      <mesh filename="file://$(find navrover_description)/meshes/right_rear_wheel_1.stl" scale="0.001 0.001 0.001"/>
-    </geometry>
-    <material name="silver"/>
-  </visual>
-  <collision>
-    <origin xyz="0.245885 0.165394 -0.063543" rpy="0 0 0"/>
-    <geometry>
-      <mesh filename="file://$(find navrover_description)/meshes/right_rear_wheel_1.stl" scale="0.001 0.001 0.001"/>
-    </geometry>
-  </collision>
-</link>
-<link name="left_front_wheel_1">
-  <inertial>
-    <origin xyz="1.5082397214483123e-07 0.05527116640249366 4.929203512721303e-07" rpy="0 0 0"/>
-    <mass value="0.737655949474422"/>
-    <inertia ixx="0.001132" iyy="0.001768" izz="0.001132" ixy="0.0" iyz="0.0" ixz="0.0"/>
-  </inertial>
-  <visual>
-    <origin xyz="-0.264518 -0.159147 -0.063543" rpy="0 0 0"/>
-    <geometry>
-      <mesh filename="file://$(find navrover_description)/meshes/left_front_wheel_1.stl" scale="0.001 0.001 0.001"/>
-    </geometry>
-    <material name="silver"/>
-  </visual>
-  <collision>
-    <origin xyz="-0.264518 -0.159147 -0.063543" rpy="0 0 0"/>
-    <geometry>
-      <mesh filename="file://$(find navrover_description)/meshes/left_front_wheel_1.stl" scale="0.001 0.001 0.001"/>
-    </geometry>
-  </collision>
-</link>
 <link name="left_front_motor_1">
   <inertial>
@@ -148,7 +86,7 @@
 <link name="right_rocker_arm_1">
   <inertial>
-    <origin xyz="3.5144696139931264e-07 0.022382973970928116 -0.019588062370497872" rpy="0 0 0"/>
-    <mass value="0.4395364357960162"/>
-    <inertia ixx="9.3e-05" iyy="0.008744" izz="0.008788" ixy="-0.0" iyz="-3e-06" ixz="-0.0"/>
+    <origin xyz="2.9281474290231146e-07 0.02209292999064974 -0.0201262955007033" rpy="0 0 0"/>
+    <mass value="0.4257120617987387"/>
+    <inertia ixx="8.7e-05" iyy="0.008739" izz="0.008786" ixy="-0.0" iyz="-1e-06" ixz="-0.0"/>
   </inertial>
   <visual>
@@ -168,7 +106,7 @@
 <link name="left_rocker_arm_1">
   <inertial>
-    <origin xyz="2.771584985891695e-07 0.018220417601364836 -0.01958806237049779" rpy="0 0 0"/>
-    <mass value="0.43953643579601614"/>
-    <inertia ixx="9.3e-05" iyy="0.008744" izz="0.008788" ixy="-0.0" iyz="4e-06" ixz="0.0"/>
+    <origin xyz="3.324283158120944e-07 0.01853003784791249 -0.02012629550070319" rpy="0 0 0"/>
+    <mass value="0.4257120617987387"/>
+    <inertia ixx="8.7e-05" iyy="0.008739" izz="0.008786" ixy="-0.0" iyz="1e-06" ixz="0.0"/>
   </inertial>
   <visual>
@@ -188,7 +126,7 @@
 <link name="rover_camera_1">
   <inertial>
-    <origin xyz="0.0035546971815331313 -2.0100020046076236e-07 0.005792514392284787" rpy="0 0 0"/>
-    <mass value="0.009136932367338056"/>
-    <inertia ixx="1e-06" iyy="0.0" izz="0.0" ixy="-0.0" iyz="-0.0" ixz="-0.0"/>
+    <origin xyz="0.003554697181533076 -2.0100020046076236e-07 0.005792514392210929" rpy="0 0 0"/>
+    <mass value="0.002153289793576474"/>
+    <inertia ixx="0.0" iyy="0.0" izz="0.0" ixy="-0.0" iyz="-0.0" ixz="-0.0"/>
   </inertial>
   <visual>
@@ -226,9 +164,69 @@
   </collision>
 </link>
+<link name="right_front_wheel_1">
+  <inertial>
+    <origin xyz="-2.4480071231791634e-06 -0.05304934910412809 3.45541559178264e-06" rpy="0 0 0"/>
+    <mass value="0.10363845671616667"/>
+    <inertia ixx="0.000149" iyy="0.000216" izz="0.000149" ixy="0.0" iyz="-0.0" ixz="-0.0"/>
+  </inertial>
+  <visual>
+    <origin xyz="-0.262818 0.165429 -0.062925" rpy="0 0 0"/>
+    <geometry>
+      <mesh filename="file://$(find navrover_description)/meshes/right_front_wheel_1.stl" scale="0.001 0.001 0.001"/>
+    </geometry>
+    <material name="silver"/>
+  </visual>
+  <collision>
+    <origin xyz="-0.262818 0.165429 -0.062925" rpy="0 0 0"/>
+    <geometry>
+      <mesh filename="file://$(find navrover_description)/meshes/right_front_wheel_1.stl" scale="0.001 0.001 0.001"/>
+    </geometry>
+  </collision>
+</link>
+<link name="right_rear_wheel_1">
+  <inertial>
+    <origin xyz="-2.1651424856328205e-06 -0.05305002932436376 3.4614773598007353e-06" rpy="0 0 0"/>
+    <mass value="0.10363845671616667"/>
+    <inertia ixx="0.000149" iyy="0.000216" izz="0.000149" ixy="0.0" iyz="-0.0" ixz="-0.0"/>
+  </inertial>
+  <visual>
+    <origin xyz="0.245885 0.165394 -0.063543" rpy="0 0 0"/>
+    <geometry>
+      <mesh filename="file://$(find navrover_description)/meshes/right_rear_wheel_1.stl" scale="0.001 0.001 0.001"/>
+    </geometry>
+    <material name="silver"/>
+  </visual>
+  <collision>
+    <origin xyz="0.245885 0.165394 -0.063543" rpy="0 0 0"/>
+    <geometry>
+      <mesh filename="file://$(find navrover_description)/meshes/right_rear_wheel_1.stl" scale="0.001 0.001 0.001"/>
+    </geometry>
+  </collision>
+</link>
+<link name="left_front_wheel_1">
+  <inertial>
+    <origin xyz="1.788549294334807e-06 0.053049405441251946 3.4614773610358585e-06" rpy="0 0 0"/>
+    <mass value="0.10363845671616667"/>
+    <inertia ixx="0.000149" iyy="0.000216" izz="0.000149" ixy="0.0" iyz="0.0" ixz="0.0"/>
+  </inertial>
+  <visual>
+    <origin xyz="-0.264518 -0.159147 -0.063543" rpy="0 0 0"/>
+    <geometry>
+      <mesh filename="file://$(find navrover_description)/meshes/left_front_wheel_1.stl" scale="0.001 0.001 0.001"/>
+    </geometry>
+    <material name="silver"/>
+  </visual>
+  <collision>
+    <origin xyz="-0.264518 -0.159147 -0.063543" rpy="0 0 0"/>
+    <geometry>
+      <mesh filename="file://$(find navrover_description)/meshes/left_front_wheel_1.stl" scale="0.001 0.001 0.001"/>
+    </geometry>
+  </collision>
+</link>
 <link name="left_rear_wheel_1">
   <inertial>
-    <origin xyz="4.3368860119796793e-07 0.0552714861822573 4.868585825046345e-07" rpy="0 0 0"/>
-    <mass value="0.737655949474422"/>
-    <inertia ixx="0.001132" iyy="0.001768" izz="0.001132" ixy="0.0" iyz="0.0" ixz="0.0"/>
+    <origin xyz="2.071413911980402e-06 0.053049725221015476 3.455415590880584e-06" rpy="0 0 0"/>
+    <mass value="0.10363845671616667"/>
+    <inertia ixx="0.000149" iyy="0.000216" izz="0.000149" ixy="0.0" iyz="0.0" ixz="0.0"/>
   </inertial>
   <visual>
@@ -246,33 +244,4 @@
   </collision>
 </link>
-<!-- <joint name="base_footprint_joint" type="fixed">
-  <origin xyz="0 0 0" rpy="0 0 0"/>
-  <parent link="base_footprint"/>
-  <child link="base_link"/>
-</joint> -->
-<joint name="right_front_wheel_joint" type="continuous">
-  <origin xyz="0.003502 -0.008922 -0.079551" rpy="0 0 0"/>
-  <parent link="right_front_motor_1"/>
-  <child link="right_front_wheel_1"/>
-  <axis xyz="0.0 1.0 0.0"/>
-  <limit effort="2.0" velocity="6.0"/>
-  <dynamics friction="0.3125" damping="0.1"/>
-</joint>
-<joint name="right_rear_wheel_joint" type="continuous">
-  <origin xyz="-0.005201 -0.008887 -0.078933" rpy="0 0 0"/>
-  <parent link="right_rear_motor_1"/>
-  <child link="right_rear_wheel_1"/>
-  <axis xyz="0.0 1.0 0.0"/>
-  <limit effort="2.0" velocity="6.0"/>
-  <dynamics friction="0.3125" damping="0.1"/>
-</joint>
-<joint name="left_front_wheel_joint" type="continuous">
-  <origin xyz="0.005202 0.008887 -0.078933" rpy="0 0 0"/>
-  <parent link="left_front_motor_1"/>
-  <child link="left_front_wheel_1"/>
-  <axis xyz="0.0 1.0 0.0"/>
-  <limit effort="2.0" velocity="6.0"/>
-  <dynamics friction="0.3125" damping="0.1"/>
-</joint>
 <joint name="left_front_motor_mount_joint" type="fixed">
   <origin xyz="0.25 0.018334 -0.030265" rpy="0 0 0"/>
@@ -301,5 +270,5 @@
   <parent link="base_link"/>
   <child link="left_rocker_arm_1"/>
-  <axis xyz="0.0 -1.0 -0.0"/>
+  <axis xyz="0.0 -1.0 0.0"/>
   <limit upper="0.261799" lower="-0.261799" effort="100" velocity="100"/>
 </joint>
@@ -313,4 +282,28 @@
   <parent link="left_rocker_arm_1"/>
   <child link="left_rear_motor_1"/>
+</joint>
+<joint name="right_front_wheel_joint" type="continuous">
+  <origin xyz="0.003502 -0.008922 -0.079551" rpy="0 0 0"/>
+  <parent link="right_front_motor_1"/>
+  <child link="right_front_wheel_1"/>
+  <axis xyz="0.0 1.0 0.0"/>
+  <limit effort="100" velocity="100"/>
+  <dynamics friction="1.0" damping="0.1"/>
+</joint>
+<joint name="right_rear_wheel_joint" type="continuous">
+  <origin xyz="-0.005201 -0.008887 -0.078933" rpy="0 0 0"/>
+  <parent link="right_rear_motor_1"/>
+  <child link="right_rear_wheel_1"/>
+  <axis xyz="0.0 1.0 0.0"/>
+  <limit effort="100" velocity="100"/>
+  <dynamics friction="1.0" damping="0.1"/>
+</joint>
+<joint name="left_front_wheel_joint" type="continuous">
+  <origin xyz="0.005202 0.008887 -0.078933" rpy="0 0 0"/>
+  <parent link="left_front_motor_1"/>
+  <child link="left_front_wheel_1"/>
+  <axis xyz="0.0 1.0 0.0"/>
+  <limit effort="100" velocity="100"/>
+  <dynamics friction="1.0" damping="0.1"/>
 </joint>
 <joint name="left_rear_wheel_joint" type="continuous">
@@ -319,6 +312,6 @@
   <child link="left_rear_wheel_1"/>
   <axis xyz="0.0 1.0 0.0"/>
-  <limit effort="2.0" velocity="6.0"/>
-  <dynamics friction="0.3125" damping="0.1"/>
+  <limit effort="100" velocity="100"/>
+  <dynamics friction="1.0" damping="0.1"/>
 </joint>
 </robot>
