Commit message: Enhance Gazebo Integration and Control for NavRover
- Added custom differential plugin (`libleo_gz_differential_plugin.so`) to improve the control of rocker arm joints. (Leo Rover Diff-sys plugin)
- Updated the `navrover.gazebo` file to include the new differential plugin, ensuring proper joint configurations for left and right rocker arms.
- Enhanced the joint state publisher configuration to include all relevant joints, ensuring accurate state reporting in Gazebo.
- Updated the `ros2_control.xacro` file to define command and state interfaces for rocker arm joints, facilitating better control through ROS 2.
- Improved bridge parameters in `bridge_parameters.yaml` to include additional topics for IMU and sensor data (LIDAR and Camera), enhancing the robot's sensor integration.
- Refined the URDF definitions in `navrover.xacro` to ensure proper mesh references and inertial properties for the rocker arms and other components.

File: navrover_control/description/ros2_contro.xacro (robot description, xacro)
@@ -1,7 +1,93 @@
 <?xml version="1.0"?>
-<robot xmls:xacro="http://www.ros.org/wiki/xacro">
+<robot xmlns:xacro="http://www.ros.org/wiki/xacro">
     <ros2_control name="GazeboSystem" type="system">
         <hardware>
             <plugin>gazebo_ros2_control::GazeboSystem</plugin>
         </hardware>
+        <!-- <joint>
+            <name>left_front_wheel_joint</name>
+            <hardwareInterface>hardware_interface/EffortJointInterface</hardwareInterface>
+        </joint>
+        <joint>
+            <name>left_rear_wheel_joint</name>
+            <hardwareInterface>hardware_interface/EffortJointInterface</hardwareInterface>
+        </joint>
+        <joint>
+            <name>right_front_wheel_joint</name>
+            <hardwareInterface>hardware_interface/EffortJointInterface</hardwareInterface>
+        </joint>
+        <joint>
+            <name>right_rear_wheel_joint</name>
+            <hardwareInterface>hardware_interface/EffortJointInterface</hardwareInterface>
+        </joint> -->
+        <!-- Define command and state interfaces -->
+        <joint>
+            <name>left_front_wheel_joint</name>
+            <!-- <hardwareInterface>hardware_interface/EffortJointInterface</hardwareInterface> -->
+            <command_interface name="velocity">
+                <param name="min">-10</param>
+                <param name="max">10</param>
+            </command_interface>
+            <state_interface name="velocity"/>
+            <state_interface name="position"/>
+            </state_interface>
+        </joint>
+        <joint>
+            <name>left_rear_wheel_joint</name>
+            <!-- <hardwareInterface>hardware_interface/EffortJointInterface</hardwareInterface> -->
+            <command_interface name="velocity">
+                <param name="min">-10</param>
+                <param name="max">10</param>
+            </command_interface>
+            <state_interface name="velocity"/>
+            <state_interface name="position"/>
+            </state_interface>
+        </joint>
+        <joint>
+            <name>right_front_wheel_joint</name>
+            <!-- <hardwareInterface>hardware_interface/EffortJointInterface</hardwareInterface> -->
+            <command_interface name="velocity">
+                <param name="min">-10</param>
+                <param name="max">10</param>
+            </command_interface>
+            <state_interface name="velocity"/>
+            <state_interface name="position"/>
+            </state_interface>
+        </joint>
+        <joint>
+            <name>right_rear_wheel_joint</name>
+            <!-- <hardwareInterface>hardware_interface/EffortJointInterface</hardwareInterface> -->
+            <command_interface name="velocity">
+                <param name="min">-10</param>
+                <param name="max">10</param>
+            </command_interface>
+            <state_interface name="velocity"/>
+            <state_interface name="position"/>
+            </state_interface>
+        </joint>
+        <joint>
+            <name>left_rocker_arm_joint</name>
+            <command_interface name="position">
+                <param name="min">-0.261799</param>
+                <param name="max">0.261799</param>
+            </command_interface>
+            <state_interface name="position"/>
+            <state_interface name="velocity"/>
+        </joint>
+        <joint>
+            <name>right_rocker_arm_joint</name>
+            <command_interface name="position">
+                <param name="min">-0.261799</param>
+                <param name="max">0.261799</param>
+            </command_interface>
+            <state_interface name="position"/>
+            <state_interface name="velocity"/>
+        </joint>
+    </ros2_control>
+     <gazebo>
+    <!-- Joint state publisher -->
+    <plugin filename="gz_ros2_control-system" name="gz_ros2_control::GazeboSimROS2ControlPlugin">
+      <parameters>$(find navrover_control)/config/navrover_controllers.yaml</parameters>
+    </plugin>
+    </gazebo>
 </robot>

File: navrover_description/urdf/navrover.xacro (robot description, xacro)
@@ -287,7 +287,6 @@
   <parent link="right_front_motor_1"/>
   <child link="right_front_wheel_1"/>
-  <axis xyz="0.0 1.0 0.0"/>
-  <limit effort="100" velocity="100"/>
-  <dynamics friction="1.0" damping="0.1"/>
+  <axis xyz="0 1 0"/>
+  <dynamics damping="0.001" friction="0.01"/>
 </joint>
 <joint name="right_rear_wheel_joint" type="continuous">
@@ -296,6 +295,5 @@
   <child link="right_rear_wheel_1"/>
   <axis xyz="0.0 1.0 0.0"/>
-  <limit effort="100" velocity="100"/>
-  <dynamics friction="1.0" damping="0.1"/>
+  <dynamics damping="0.001" friction="0.01"/>
 </joint>
 <joint name="left_front_wheel_joint" type="continuous">
@@ -304,6 +302,5 @@
   <child link="left_front_wheel_1"/>
   <axis xyz="0.0 1.0 0.0"/>
-  <limit effort="100" velocity="100"/>
-  <dynamics friction="1.0" damping="0.1"/>
+  <dynamics damping="0.001" friction="0.01"/>
 </joint>
 <joint name="left_rear_wheel_joint" type="continuous">
@@ -312,6 +309,5 @@
   <child link="left_rear_wheel_1"/>
   <axis xyz="0.0 1.0 0.0"/>
-  <limit effort="100" velocity="100"/>
-  <dynamics friction="1.0" damping="0.1"/>
+  <dynamics damping="0.001" friction="0.01"/>
 </joint>
 </robot>
