Commit message: Update package dependencies and controller configuration

File: navrover_control/description/ros2_control.xacro (robot description, xacro)
@@ -6,8 +6,8 @@
         </hardware>
         <!-- Define command and state interfaces -->
-        <joint name = "left_front_wheel_joint">
+        <!-- <joint name = "left_front_wheel_joint">
             <command_interface name="velocity">
-                <param name="min">-1.5</param>  <!-- Adjusted min value based on velocity -->
-                <param name="max">1.5</param>    <!-- Adjusted max value based on velocity -->
+                <param name="min">-1.5</param>
+                <param name="max">1.5</param>
             </command_interface>
             <state_interface name="velocity"/>
@@ -16,6 +16,6 @@
         <joint name = "left_rear_wheel_joint">
             <command_interface name="velocity">
-                <param name="min">-1.5</param>  <!-- Adjusted min value based on velocity -->
-                <param name="max">1.5</param>    <!-- Adjusted max value based on velocity -->
+                <param name="min">-1.5</param>
+                <param name="max">1.5</param>
             </command_interface>
             <state_interface name="velocity"/>
@@ -24,6 +24,6 @@
         <joint name = "right_front_wheel_joint">
             <command_interface name="velocity">
-                <param name="min">-1.5</param>  <!-- Adjusted min value based on velocity -->
-                <param name="max">1.5</param>    <!-- Adjusted max value based on velocity -->
+                <param name="min">-1.5</param>
+                <param name="max">1.5</param>
             </command_interface>
             <state_interface name="velocity"/>
@@ -32,30 +32,29 @@
         <joint name = "right_rear_wheel_joint">
             <command_interface name="velocity">
-                <param name="min">-1.5</param>  <!-- Adjusted min value based on velocity -->
-                <param name="max">1.5</param>    <!-- Adjusted max value based on velocity -->
+                <param name="min">-1.5</param>
+                <param name="max">1.5</param>
             </command_interface>
             <state_interface name="velocity"/>
             <state_interface name="position"/>
-        </joint>
+        </joint> -->
         <joint name = "left_rocker_arm_joint">
             <command_interface name="effort">
-                <param name="min">-0.261799</param>
-                <param name="max">0.261799</param>
+                <param name="min">-0.24</param>
+                <param name="max">0.24</param>
             </command_interface>
-            <state_interface name="position"/>
+            <state_interface name="effort"/>
         </joint>
         <joint name = "right_rocker_arm_joint">
             <command_interface name="effort">
-                <param name="min">-0.261799</param>
-                <param name="max">0.261799</param>
+                <param name="min">-0.24</param>
+                <param name="max">0.24</param>
             </command_interface>
-            <state_interface name="position"/>
+            <state_interface name="effort"/>
         </joint>
     </ros2_control>
   <gazebo>
     <!-- Joint state publisher -->
-    <plugin filename="libgz_ros2_control-system.so" name="gz_ros2_control::GazeboSimROS2ControlPlugin">
+    <plugin filename="libgz_ros2_control-system" name="gz_ros2_control::GazeboSimROS2ControlPlugin">
       <parameters>$(find navrover_control)/config/navrover_controllers.yaml</parameters>
-      <controller_manager_prefix_node_name>controller_manager</controller_manager_prefix_node_name>
     </plugin>
   </gazebo>

File: navrover_description/urdf/navrover.xacro (robot description, xacro)
@@ -264,6 +264,7 @@
   <parent link="base_link"/>
   <child link="right_rocker_arm_1"/>
-  <axis xyz="0.0 -1.0 0.0"/>
+  <axis xyz="0.0 1.0 0.0"/>
   <limit upper="0.261799" lower="-0.261799" effort="100" velocity="100"/>
+  <!-- <dynamics friction = "1.0" damping = "0.1"/> -->
 </joint>
 <joint name="left_rocker_arm_joint" type="revolute">
@@ -271,6 +272,7 @@
   <parent link="base_link"/>
   <child link="left_rocker_arm_1"/>
-  <axis xyz="0.0 -1.0 0.0"/>
+  <axis xyz="0.0 1.0 0.0"/>
   <limit upper="0.261799" lower="-0.261799" effort="100" velocity="100"/>
+  <!-- <dynamics friction = "1.0" damping = "0.1"/> -->
 </joint>
 <joint name="rover_front_camera_joint" type="fixed">

Commit message: Implement PID Controllers for Rocker Arms
- Updated navrover_controllers.yaml to define left and right rocker position controllers using JointGroupPositionController.
- Modified ros2_control.xacro to include command and state interfaces for left and right rocker arms.
- Enhanced gazebo.launch.py to spawn the rocker position controllers with the appropriate parameters.
- Ensured joint state publisher includes rocker arms in the Gazebo simulation.
- Implemented Gazebo Sim Joint Position Controller System

File: navrover_control/description/ros2_control.xacro (robot description, xacro)
@@ -39,16 +39,20 @@
         </joint> -->
         <joint name = "left_rocker_arm_joint">
-            <command_interface name="effort">
-                <param name="min">-0.24</param>
-                <param name="max">0.24</param>
+            <command_interface name="position">
+                <param name="min">-0.261799</param>
+                <param name="max">0.261799</param>
             </command_interface>
             <state_interface name="effort"/>
+            <state_interface name="position"/>
+            <state_interface name="velocity"/>
         </joint>
         <joint name = "right_rocker_arm_joint">
-            <command_interface name="effort">
-                <param name="min">-0.24</param>
-                <param name="max">0.24</param>
+            <command_interface name="position">
+                <param name="min">-0.261799</param>
+                <param name="max">0.261799</param>
             </command_interface>
             <state_interface name="effort"/>
+            <state_interface name="position"/>
+            <state_interface name="velocity"/>
         </joint>
     </ros2_control>
@@ -58,4 +62,20 @@
       <parameters>$(find navrover_control)/config/navrover_controllers.yaml</parameters>
     </plugin>
+    <!-- Gz Sim Joint Position Controller System-->
+    <plugin filename="gz-sim-joint-position-controller-system" name="gz::sim::systems::JointPositionController">
+        <joint_name>left_rocker_arm_joint</joint_name>
+        <topic>/left_rocker_position_controller/commands</topic>
+        <p_gain>8.0</p_gain>
+        <i_gain>5.0</i_gain>
+        <d_gain>5.0</d_gain>
+    </plugin>
+    <!-- Gz Sim Joint Position Controller System-->
+    <plugin filename="gz-sim-joint-position-controller-system" name="gz::sim::systems::JointPositionController">
+        <joint_name>right_rocker_arm_joint</joint_name>
+        <topic>/right_rocker_position_controller/commands</topic>
+        <p_gain>8.0</p_gain>
+        <i_gain>5.0</i_gain>
+        <d_gain>5.0</d_gain>
+    </plugin>
   </gazebo>
 </robot>

File: navrover_description/urdf/navrover.xacro (robot description, xacro)
@@ -266,5 +266,5 @@
   <axis xyz="0.0 1.0 0.0"/>
   <limit upper="0.261799" lower="-0.261799" effort="100" velocity="100"/>
-  <!-- <dynamics friction = "1.0" damping = "0.1"/> -->
+  <dynamics friction = "1.0" damping = "0.1"/>
 </joint>
 <joint name="left_rocker_arm_joint" type="revolute">
@@ -274,5 +274,5 @@
   <axis xyz="0.0 1.0 0.0"/>
   <limit upper="0.261799" lower="-0.261799" effort="100" velocity="100"/>
-  <!-- <dynamics friction = "1.0" damping = "0.1"/> -->
+  <dynamics friction = "1.0" damping = "0.1"/>
 </joint>
 <joint name="rover_front_camera_joint" type="fixed">
